File: DCR_MainBoard/DCR_MainBoard.kicad_sch (KiCad schematic)
At the start: 32 parts, among them J1 ANT, J3 LO, J4 PWR, J5 Audio, U1 QPR_Filter, U2 SA612, U3 LM7806, U4 LM386

Commit message: Update snapada
Parts:
- added C8: 100n, Capacitor_SMD:C_1206_3216Metric, symbol Device:C
- added H1, H2, H3, H4: MountingHole, MountingHole:MountingHole_3.2mm_M3, symbol Mechanical:MountingHole
- added TP1: TP1, TestPoint:TestPoint_THTPad_1.0x1.0mm_Drill0.5mm, symbol Connector:TestPoint
- added TP2: TP2, TestPoint:TestPoint_THTPad_1.0x1.0mm_Drill0.5mm, symbol Connector:TestPoint
- added TP3: TP3, TestPoint:TestPoint_THTPad_1.0x1.0mm_Drill0.5mm, symbol Connector:TestPoint
- added TP4: TP4, TestPoint:TestPoint_THTPad_1.0x1.0mm_Drill0.5mm, symbol Connector:TestPoint
- added TP5: TP5, TestPoint:TestPoint_THTPad_1.0x1.0mm_Drill0.5mm, symbol Connector:TestPoint
- added TP6: TP6, TestPoint:TestPoint_THTPad_1.0x1.0mm_Drill0.5mm, symbol Connector:TestPoint
Connections:
- net at C4.1, R1.2, U4.3 (+): now also TP4.1
- net at C15.1, R8.2, U4.5: now also TP6.1
- net at J1.1, J1.2, U1.1 (IN)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: now also TP1.1
- net at C1.1, C3.1, U2.4 (OUT_A): now also TP3.1
- net at U1.7 (OUT), U1.8 (OUT): now also C8.1; no longer U2.1 (IN_A)
- net at C6.2, U2.6 (OSC_B): now also TP5.1
- new net: C8.2, TP2.1, U2.1 (IN_A)
