File: DCR_MainBoard/DCR_MainBoard.kicad_pcb (KiCad board)
At the start: 2 copper layers, 97.7 x 59.7 mm, 32 parts, among them J1 ANT, J3 LO SMA, J4 PWR, J5 Audio, U1 QPR_Filter, U2 SA612, U3 LM7806, U4 LM386

Commit message: Update snapada
Parts:
- added C8: 100n, Capacitor_SMD:C_1206_3216Metric, F.Cu at (43.6, 44.3)
- added H1: MountingHole, MountingHole:MountingHole_3.2mm_M3, F.Cu at (25.7, 27.1)
- added H2: MountingHole, MountingHole:MountingHole_3.2mm_M3, F.Cu at (25.7, 78.7)
- added H3: MountingHole, MountingHole:MountingHole_3.2mm_M3, F.Cu at (115.4, 78.6)
- added H4: MountingHole, MountingHole:MountingHole_3.2mm_M3, F.Cu at (115.5, 27.3)
- added TP1: TP1, TestPoint:TestPoint_THTPad_1.0x1.0mm_Drill0.5mm, F.Cu at (34.2, 30.5)
- added TP2: TP2, TestPoint:TestPoint_THTPad_1.0x1.0mm_Drill0.5mm, F.Cu at (49.5, 41.4)
- added TP3: TP3, TestPoint:TestPoint_THTPad_1.0x1.0mm_Drill0.5mm, F.Cu at (54.0, 59.2)
- added TP4: TP4, TestPoint:TestPoint_THTPad_1.0x1.0mm_Drill0.5mm, F.Cu at (66.4, 72.0)
- added TP5: TP5, TestPoint:TestPoint_THTPad_1.0x1.0mm_Drill0.5mm, F.Cu at (60.6, 50.0)
- added TP6: TP6, TestPoint:TestPoint_THTPad_1.0x1.0mm_Drill0.5mm, F.Cu at (82.6, 78.6)
- J3: value LO SMA -> LO
- moved J1 20.2 mm to (50.2, 36.5)
- moved C2 15.4 mm to (45.1, 48.8)
- moved U2 15.4 mm to (48.4, 45.0)
- moved C5 15.4 mm to (54.8, 41.7)
- moved R2 15.4 mm to (59.6, 41.7)
- moved C1 15.4 mm to (46.9, 55.6)
- moved C3 15.4 mm to (48.7, 61.1)
- moved D1 9.09 mm to (115.3, 39.1), turned to 90 degrees
- moved U1 7.31 mm to (29.0, 45.5)
Connections:
- U2 pad 1: Net-(U1-Pad7) -> Net-(U2-Pad1)
Routing:
- net Net-(U1-Pad7): track 57.1 -> 33.1 mm
- net RX6V: track 66.8 -> 48.4 mm
- net Net-(C3-Pad2): track 30.1 -> 14.9 mm
- net Net-(J1-Pad1): track 11.5 -> 23.7 mm
- net Net-(C4-Pad1): track 5.40 -> 16.1 mm
- net Net-(C6-Pad2): track 21.0 -> 31.3 mm
- net Net-(U2-Pad1): track 0.00 -> 8.01 mm
- net Net-(C15-Pad1): track 10.9 -> 17.3 mm
- net Net-(C1-Pad1): track 11.7 -> 17.8 mm
- net Net-(D1-Pad2): track 2.86 -> 0.00 mm

Commit message: VE3POA Update & Gerbers
Routing:
- net Net-(D1-Pad2): track 0.00 -> 4.17 mm
