File: DCV V2/DCV v2.kicad_sch (KiCad schematic)
At the start: 44 parts, among them J1 ANT, J10 TP3, J2 TP6, J3 LO, J4 PWR, J5 Audio, J6 TP1, J7 TP2, J8 TP5, J9 TP4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

Commit message: Added_Version_2
Other:
- note removed: "CP-002A-ND Power barrel connector 486-3417-ND 3.5mm mono phone jack CON-SMA-EDGE-S-ND CONN SMA JACK STR EDGE MNT A97553-ND CONN BNC JACK R/A 50 OHM PCB PTV09A-2020F-A103-ND POT 10K OHM 1/20W CARBON LOG"
Changed lines of the file:
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@@
     (stroke (width 0) (type default) (color 0 0 0 0))
-  )
-  (text "CP-002A-ND             Power barrel connector\n486-3417-ND            3.5mm mono phone jack\nCON-SMA-EDGE-S-ND      CONN SMA JACK STR EDGE MNT\nA97553-ND              CONN BNC JACK R/A 50 OHM PCB\nPTV09A-2020F-A103-ND   POT 10K OHM 1/20W CARBON LOG"
-    (at 185.42 48.26 0)
-    (effects (font (size 1.27 1.27)) (justify left bottom))
   )
   (global_label "12V" (shape output) (at 20.955 23.495 90) (fields_autoplaced)
