File: DCR V2/DCR v2.kicad_pcb (KiCad board)
At the start: 2 copper layers, 97.7 x 59.7 mm, 45 parts, among them J1 ANT, J10 TP3, J2 TP6, J3 LO, J4 PWR, J5 Audio, J6 TP1, J7 TP2, J8 TP5, J9 TP4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

Commit message: 7896 Update
Parts:
- U3: value 78L06 -> L78L06; footprint Package_TO_SOT_THT:TO-92L_Inline_Wide -> Package_TO_SOT_THT:TO-92_Inline
- moved U3 3.39 mm to (181.2, 80.4), turned to 90 degrees
- moved C10 0.84 mm to (177.0, 82.5)
Connections:
- U3 pad 1: 12V -> RX6V
- U3 pad 3: RX6V -> 12V
Routing:
- net RX6V: track 50.7 -> 57.4 mm
- net 12V: track 63.9 -> 61.2 mm
